File: Stage1 - STM/voxboard/voxboard.kicad_sch (KiCad schematic)
At the start: 0 parts

Commit message: Assets
Parts:
- added C1, C20, C30, C31, C32, C33, C34, C4, C7: 100n, symbol Device:C
- added C13, C14, C29: 10u, symbol Device:C
- added C15: 1n2, symbol Device:C
- added C16: 10p, symbol Device:C
- added C17: 8n2, symbol Device:C
- added C18, C19: 47u, symbol Device:C
- added C2, C3: 1u, symbol Device:C
- added C21, C22: 4u7, symbol Device:C
- added C24: 1000u, symbol Device:C_Polarized
- added C5, C6: 16p, symbol Device:C
- added D1: D_Zener, symbol Device:D_Zener
- added D2: 40V, symbol Device:D_Schottky
- added D3: RED, symbol Device:LED
- added D4: SMAJ43A, Diode_SMD:D_SMA, symbol Diode:SMAJ43A
- added F1: Fuse, symbol Device:Fuse
- added FB2, FB3: FerriteBead, symbol Device:FerriteBead
- added IC1: TPS54331DR, SOIC127P600X175-8N, symbol TPS54331DR:TPS54331DR
- added L1: 8u2, symbol Device:L
- added P2: USB_C_Plug_USB2.0, symbol Connector:USB_C_Plug_USB2.0
- added PS2: XT60PW-M, XT60PWM, symbol XT60PW-M:XT60PW-M
- added Q2, Q3: PMOS, symbol Simulation_SPICE:PMOS
- added R1: 5k1, symbol Device:R
- added R18, R19: 1k, symbol Device:R
- added R2: 25k, symbol Device:R
- added R26, R8: 10k, symbol Device:R
- added R27: 100k, symbol Device:R
- added R3: 10k5, symbol Device:R
- added R4: 2k, symbol Device:R
- added R5: 1k5, symbol Device:R
- added SW2: SW_Push, symbol Switch:SW_Push
- added SW3: SW_SPDT, symbol Switch:SW_SPDT
- added TP3, TP4, TP5: TestPoint, symbol Connector:TestPoint
- added U1: STM32F446RETx, Package_QFP:LQFP-64_10x10mm_P0.5mm, symbol MCU_ST_STM32F4:STM32F446RETx
- added U2: AP7361C-33Y5-13, SOT89-5_DIO, symbol AP7361C-33Y5-13:AP7361C-33Y5-13
- added U3: SN65HVD230DR, D8, symbol SN65HVD230DR:SN65HVD230DR
- added U4: USBLC6-2SC6, Package_TO_SOT_SMD:SOT-23-6, symbol Power_Protection:USBLC6-2SC6
- added Y1: 8MHz, symbol Device:Crystal_GND24
Connections:
- new net: R19.2, U1.16 (PA2)
- new net: C20.1, IC1.1 (BOOT)
- new net: C20.2, D2.1 (K), IC1.8 (PH), L1.1
- new net: D1.1 (K), F1.2, Q2.3 (S)
- new net: D1.2 (A), Q2.2 (G), R8.2
- new net: FB3.2, PS2.2 (-), TP4.1
- new net: F1.1, PS2.1 (+), TP5.1
- new net: C17.1, IC1.4 (SS)
- new net: IC1.5 (VSENSE), R3.2, R4.1
- new net: C16.1, IC1.6 (COMP), R2.1
- new net: P2.A5 (CC), R1.1
- new net: R18.2, U1.42 (PA9)
- new net: C7.1, Q3.2 (G), R27.2
- new net: C15.1, R2.2
- new net: D3.1 (K), R5.1
- new net: R26.1, SW3.2 (B)
- new net +24V: C13.1, C14.1, C24.1, D4.1 (A1), IC1.2 (VIN), Q2.1 (D)
- new net +3.3V: C1.1, C13.2, C14.2, C15.2, C16.2, C17.2, C18.2, C19.2, C2.1, C2.2, C21.2, C22.1, C22.2, C24.2, C29.1, C29.2, C3.2, C30.1, C30.2, C31.1, C31.2, C32.1, C32.2, C33.1, C33.2, C34.1, C34.2, C4.2, C5.2, C6.2, D2.2 (A), D3.2 (A), D4.2 (A2), FB2.2, FB3.1, IC1.7 (GND), P2.A1 (GND), P2.A12 (GND), P2.B1 (GND), P2.B12 (GND), R1.2, R4.2, R5.2, R8.1, SW2.1, SW3.1 (A), SW3.3 (C), U1.1 (VBAT), U1.12 (VSSA), U1.18 (VSS), U1.19 (VDD), U1.31 (VSS), U1.32 (VDD), U1.47 (VSS), U1.48 (VDD), U1.63 (VSS), U1.64 (VDD), U2.2 (GND), U2.5 (OUT), U3.2 (GND), U3.3 (VCC), U4.2 (GND), Y1.2 (G), Y1.4 (G)
- new net +3.3VA: C3.1, C4.1, FB2.1, U1.13 (VDDA)
- new net +5V: C18.1, C19.1, C21.1, L1.2, Q3.1 (D), R27.1, R3.1, TP3.1, U2.1 (EN), U2.4 (IN)
- new net BOOT_BTN: R26.2, U1.60 (BOOT0)
- new net CAN1_RX: U1.61 (PB8), U3.1 (D)
- new net CAN1_TX: U1.62 (PB9), U3.4 (R)
- new net CAN2_RX: U1.33 (PB12)
- new net CAN2_TX: U1.34 (PB13)
- new net I2C_SCL: U1.29 (PB10)
- new net I2C_SDA: U1.53 (PC12)
- new net NRST: C1.2, SW2.2, U1.7 (NRST)
- new net OSC_IN: C5.1, U1.5 (PH0), Y1.1
- new net OSC_OUT: C6.1, U1.6 (PH1), Y1.3
- new net SPI1_MISO: U1.22 (PA6)
- new net SPI1_MOSI: U1.23 (PA7)
- new net SPI1_SCK: U1.21 (PA5)
- new net SPI2_MISO: U1.35 (PB14)
- new net SPI2_MOSI: U1.36 (PB15)
- new net SPI2_SCK: U1.38 (PC7)
- new net STEP_MOT_SPI_00: U1.14 (PA0)
- new net STEP_MOT_SPI_01: U1.37 (PC6)
- new net STEP_MOT_U1_00: U1.41 (PA8)
- new net STEP_MOT_U1_01: U1.56 (PB4)
- new net STEP_MOT_U2_00: U1.50 (PA15)
- new net STEP_MOT_U2_01: U1.58 (PB6)
- new net SWCLK: U1.49 (PA14)
- new net SWDIO: U1.46 (PA13)
- new net SWO: U1.55 (PB3)
- new net UARTTX_MOT_U1: R18.1
- new net UARTTX_MOT_U2: R19.1
- new net USB_D+: P2.A6 (D+), U1.45 (PA12), U4.1 (I/O1), U4.6 (I/O1)
- new net USB_D-: P2.A7 (D-), U1.44 (PA11), U4.3 (I/O2), U4.4 (I/O2)
- new net VBUS: C7.2, P2.A4 (VBUS), P2.A9 (VBUS), P2.B4 (VBUS), P2.B9 (VBUS), Q3.3 (S), U4.5 (VBUS)
- no-connect marks 0 -> 6
Other:
- added sheet MOTOR_CONTROL (motors_voxboard.kicad_sch)
- note added: "24V -> 5V/3A Buck Convertor"
- note added: "24V INPUT XT60"
- note added: "3.3V VDD/VBAT"
- note added: "3.3VA VDDA"
- note added: "5V -> 3.3V/1A Voltage Regulator (LDO)"
- note added: "5V/VBUS"
- note added: "BOOT"
- note added: "CRYSTAL RESONATOR"
- note added: "ESD USBLC6-2SC6"
- note added: "NRST"
- note added: "USBC 2.0"
