File: Stage1 - STM/voxboard/voxboard.kicad_sch (KiCad schematic)
At the start: 57 parts, among them IC1 TPS54331DR, P2 USB_C_Plug_USB2.0, Q2 PMOS, Q3 PMOS, SW2 SW_Push, SW3 SW_SPDT, U1 STM32F446RETx, U2 AP7361C-33Y5-13, U3 SN65HVD230DR, U4 USBLC6-2SC6, Y1 8MHz

Commit message: Updates 01
Parts:
- removed FB3: FerriteBead, symbol Device:FerriteBead
- removed IC1: TPS54331DR, SOIC127P600X175-8N, symbol TPS54331DR:TPS54331DR
- removed P2: USB_C_Plug_USB2.0, symbol Connector:USB_C_Plug_USB2.0
- removed PS2: XT60PW-M, XT60PWM, symbol XT60PW-M:XT60PW-M
- removed Q3: PMOS, symbol Simulation_SPICE:PMOS
- removed U1: STM32F446RETx, Package_QFP:LQFP-64_10x10mm_P0.5mm, symbol MCU_ST_STM32F4:STM32F446RETx
- removed U2: AP7361C-33Y5-13, SOT89-5_DIO, symbol AP7361C-33Y5-13:AP7361C-33Y5-13
- removed U3: SN65HVD230DR, D8, symbol SN65HVD230DR:SN65HVD230DR
- removed U4: USBLC6-2SC6, Package_TO_SOT_SMD:SOT-23-6, symbol Power_Protection:USBLC6-2SC6
- added C10, C12, C23, C26, C37, C38, C40, C41, C43, C44, C46, C47, C49, C50: 100n, Capacitor_SMD:C_0402_1005Metric, symbol Device:C
- added C11, C35: 4n7, Capacitor_SMD:C_0402_1005Metric, symbol Device:C
- added C25: 10u, Capacitor_SMD:C_0603_1608Metric, symbol Device:C
- added C27: 4u7, Capacitor_SMD:C_0603_1608Metric, symbol Device:C
- added C28, C36, C8, C9: 100p, Capacitor_SMD:C_0402_1005Metric, symbol Device:C
- added C39, C52: 220u, Capacitor_THT:CP_Radial_D10.0mm_P5.00mm, symbol Device:C_Polarized
- added C42, C45, C48, C51: 100u, Capacitor_THT:CP_Radial_D8.0mm_P3.50mm, symbol Device:C_Polarized
- added CR2: PESD2CANFD24V-TR, Package_TO_SOT_SMD:SOT-23, symbol Arsenal_Lib:PESD2CANFD24V-TR
- added D10, D5: YELLOW, LED_SMD:LED_0603_1608Metric, symbol Device:LED
- added D6: RED, LED_SMD:LED_0603_1608Metric, symbol Device:LED
- added D7: YELLOW, LED_SMD:LED_0805_2012Metric, symbol Device:LED
- added D8: 24V/5V, Diode_SMD:D_SMC, symbol Device:D_Schottky
- added DRIVER1, DRIVER2, DRIVER3, DRIVER4: TMC2209, Arsenal_Lib:MODULE_TMC2209_5160, symbol Arsenal_Lib:TMC2209
- added DRIVER5, DRIVER6: TMC5160, Arsenal_Lib:MODULE_TMC2209_5160, symbol Arsenal_Lib:TMC5160
- added FB1: 600R, Inductor_SMD:L_1210_3225Metric, symbol Device:FerriteBead
- added IC1: TPS54331DR, Package_SO:SOIC-8_3.9x4.9mm_P1.27mm, symbol Arsenal_Lib:TPS54331DR
- added J1: USB4110-GF-A, Arsenal_Lib:USB_C_Receptacle_GCT_USB4110, symbol Arsenal_Lib:USB4110-GF-A
- added J11, J12, J13, J14, J15, J16, J17, J18: Conn_01x04_Pin, Arsenal_Lib:JST_GH_BM04B-GHS-TBT_1x04-1MP_P1.25mm_Vertical, symbol Connector:Conn_01x04_Pin
- added JC1, JC2, JC3: Conn_01x03_Pin, Arsenal_Lib:JST_GH_BM03B-GHS-TBT_1x03-1MP_P1.25mm_Vertical, symbol Connector:Conn_01x03_Pin
- added JM1, JM2, JM3, JM4, JM5, JM6: Conn_01x04_Pin, Arsenal_Lib:JST_VH_B4P-VH-FB-B_1x04_P3.96mm_Vertical, symbol Connector:Conn_01x04_Pin
- added JS1: Conn_01x05_Pin, Arsenal_Lib:PinHeader_1x05_P2.54mm_Vertical, symbol Connector:Conn_01x05_Pin
- added JU1: Conn_01x03_Pin, Connector_PinHeader_2.54mm:PinHeader_1x03_P2.54mm_Vertical, symbol Connector:Conn_01x03_Pin
- added PS1: XT60PW-M, Arsenal_Lib:AMASS_XT60PW-M_1x02_P7.20mm_Horizontal, symbol Arsenal_Lib:XT60PW-M
- added Q1: PMOS, Package_TO_SOT_SMD:SOT-23, symbol Simulation_SPICE:PMOS
- added R10, R12, R13, R14, R16, R17, R24, R25, R32, R33, R37, R39, R40, R41, R42, R43, R44, R45, R46, R47, R6, R9: 33o, Resistor_SMD:R_0402_1005Metric, symbol Device:R
- added R11, R15, R28, R30, R31, R34, R38, R48, R49, R53, R7: 10k, Resistor_SMD:R_0402_1005Metric, symbol Device:R
- added R20, R21, R22, R23: 60, Resistor_SMD:R_0603_1608Metric, symbol Device:R
- added R29: 5k1, Resistor_SMD:R_0402_1005Metric, symbol Device:R
- added R35, R36: 4k7, Resistor_SMD:R_0402_1005Metric, symbol Device:R
- added R50, R52: 220, Resistor_SMD:R_0402_1005Metric, symbol Device:R
- added R51: 3k, Resistor_SMD:R_0402_1005Metric, symbol Device:R
- added TP1, TP2: TestPoint, TestPoint:TestPoint_Pad_2.0x2.0mm, symbol Connector:TestPoint
- added TP6: TestPoint, TestPoint:TestPoint_Pad_D2.0mm, symbol Connector:TestPoint
- added U1: STM32F446RETx, Arsenal_Lib:LQFP64-10x10mm, symbol Arsenal_Lib:STM32F446RETx
- added U11: SN65HVD230DR, Package_SO:SOIC-8_3.9x4.9mm_P1.27mm, symbol Arsenal_Lib:SN65HVD230DR
- added U12, U3: TPD4E02B04DQAR, Package_SON:USON-10_2.5x1.0mm_P0.5mm, symbol Arsenal_Lib:TPD4E02B04DQAR
- added U14, U15: PESD5V0F1BRSFYL, Diode_SMD:Nexperia_DSN0603-2_0.6x0.3mm_P0.4mm, symbol Arsenal_Lib:PESD5V0F1BRSFYL
- added U16, U4: SM12OC, Package_TO_SOT_SMD:SOT-23, symbol Arsenal_Lib:ESD122DMXR
- added U18, U19, U20, U21, U22, U6: MT6835, Connector_JST:JST_GH_BM07B-GHS-TBT_1x07-1MP_P1.25mm_Vertical, symbol Arsenal_Lib:MT6835
- added U2: AP7361C-33Y5-13, Arsenal_Lib:AP7361C-33Y5-13_SOT89-5_DIO, symbol Arsenal_Lib:AP7361C-33Y5-13
- added U5: TPD2E1B06DRLR, Package_TO_SOT_SMD:SOT-666, symbol Arsenal_Lib:TPD2E1B06DRLR
- C1, C30, C31, C32, C33, C34, C4: footprint (none) -> Capacitor_SMD:C_0402_1005Metric
- C13, C14, C18, C19: footprint (none) -> Capacitor_SMD:C_1210_3225Metric
- C15, C16, C20: footprint (none) -> Capacitor_SMD:C_0805_2012Metric
- C17: footprint (none) -> Capacitor_SMD:C_0201_0603Metric
- C2, C21, C22, C29, C3: footprint (none) -> Capacitor_SMD:C_0603_1608Metric
- C24: footprint (none) -> Capacitor_THT:CP_Radial_D8.0mm_P3.50mm
- C5, C6: value 16p -> 14p; footprint (none) -> Capacitor_SMD:C_0402_1005Metric
- C7: value 100n -> 10u; footprint (none) -> Capacitor_SMD:C_0603_1608Metric
- D1: footprint (none) -> Diode_SMD:D_SOD-123
- D2: footprint (none) -> Diode_SMD:D_SMA
- D3: value RED -> YG; footprint (none) -> LED_SMD:LED_0603_1608Metric
- D4: value SMAJ43A -> SMAJ26A
- F1: footprint (none) -> Arsenal_Lib:CONN_3557-2_KEY
- FB2: value FerriteBead -> 120R; footprint (none) -> Inductor_SMD:L_0603_1608Metric
- L1: footprint (none) -> Arsenal_Lib:L_KOHERELEC_MDA7050_7.3x6.6mm
- Q2: footprint (none) -> Package_TO_SOT_SMD:TO-252-2
- R1, R18, R19, R2, R26, R3, R4, R8: footprint (none) -> Resistor_SMD:R_0402_1005Metric
- R27: value 100k -> 220; footprint (none) -> Resistor_SMD:R_0402_1005Metric
- R5: value 1k5 -> 220; footprint (none) -> Resistor_SMD:R_0402_1005Metric
- SW2: footprint (none) -> Arsenal_Lib:SW_PUSH_B3U-1000PM
- SW3: footprint (none) -> Button_Switch_SMD:SW_SPDT_PCM12
- TP3, TP5: footprint (none) -> TestPoint:TestPoint_Pad_D2.0mm
- TP4: footprint (none) -> TestPoint:TestPoint_Pad_2.0x2.0mm
- Y1: footprint (none) -> Arsenal_Lib:Crystal_SMD_3225-4Pin_3.2x2.5mm
Connections:
- net +24V: now also C7.2, TP5.1, C23.1, C37.1, C38.2, C39.1, C41.1, C42.1, C44.1, C45.1, C47.1, C48.1, C50.1, C51.1, C52.1, D6.2 (A), DRIVER1.8 (VM), DRIVER2.8 (VM), DRIVER3.8 (VM), DRIVER4.8 (VM), DRIVER5.8 (VM), DRIVER6.8 (VM), IC1.2 (VIN)
- net +3.3V: now also C10.1, C12.1, C25.1, C26.1, C40.1, C43.1, C46.1, C49.1, DRIVER1.2 (VDD), DRIVER2.15 (MS1), DRIVER2.2 (VDD), DRIVER3.2 (VDD), DRIVER4.15 (MS1), DRIVER4.2 (VDD), DRIVER5.2 (VDD), DRIVER6.2 (VDD), J11.1 (Pin_1), J12.1 (Pin_1), J13.1 (Pin_1), J14.1 (Pin_1), J15.1 (Pin_1), J16.1 (Pin_1), J17.1 (Pin_1), J18.1 (Pin_1), JS1.1 (Pin_1), R11.2, R15.2, R28.2, R30.2, R34.2, R35.1, R36.2, R38.2, R48.2, R49.2, R7.2, TP6.1, U1.1 (VBAT), U1.19 (VDD), U1.32 (VDD), U1.48 (VDD), U1.64 (VDD), U11.3 (VCC), U2.5 (OUT); no longer C1.1, C13.2, C14.2, C15.2, C16.2, C17.2, C18.2, C19.2, C2.2, C21.2, C22.2, C24.2, C29.2, C3.2, C30.2, C31.2, C32.2, C33.2, C34.2, C4.2, C5.2, C6.2, D2.2 (A), D4.2 (A2), R1.2, R4.2, R5.2, R8.1, SW2.1, SW3.1 (A), Y1.2 (G), Y1.4 (G)
- net +3.3VA: now also U1.13 (VDDA)
- net +5V: now also D8.1 (K), Q1.1 (D), U2.1 (EN), U2.4 (IN); no longer C18.1, C19.1, L1.2, R27.1, R3.1, TP3.1
- net BOOT_BTN: now also U1.60 (BOOT0)
- net CAN1_RX: now also U1.61 (PB8), U11.1 (D)
- net CAN1_TX: now also U1.62 (PB9), U11.4 (R)
- net I2C_SCL: now also R24.1, R35.2, U1.29 (PB10)
- net I2C_SDA: now also R25.1, R36.1, U1.53 (PC12)
- net NRST: now also JS1.5 (Pin_5), U1.7 (NRST)
- net OSC_IN: now also U1.5 (PH0)
- net OSC_OUT: now also U1.6 (PH1)
- net SPI1_MISO: now also DRIVER5.12 (SDO), DRIVER6.12 (SDO), U1.22 (PA6), U12.2 (D1-), U12.9 (NC)
- net SPI1_MOSI: now also DRIVER5.15 (SDI), DRIVER6.15 (SDI), U1.23 (PA7), U12.1 (D1+), U12.10 (NC)
- net SPI1_SCK: now also DRIVER5.14 (SCK), DRIVER6.14 (SCK), U1.21 (PA5), U12.4 (D2+), U12.7 (NC)
- net SPI2_MISO: now also U1.35 (PB14), U18.3 (MISO), U19.3 (MISO), U20.3 (MISO), U21.3 (MISO), U22.3 (MISO), U3.2 (D1-), U3.9 (NC), U6.3 (MISO)
- net SPI2_MOSI: now also U1.36 (PB15), U18.4 (MOSI), U19.4 (MOSI), U20.4 (MOSI), U21.4 (MOSI), U22.4 (MOSI), U3.4 (D2+), U3.7 (NC), U6.4 (MOSI)
- net SPI2_SCK: now also U1.34 (PB13), U18.5 (SCK), U19.5 (SCK), U20.5 (SCK), U21.5 (SCK), U22.5 (SCK), U3.1 (D1+), U3.10 (NC), U6.5 (SCK)
- net STEP_MOT_SPI_00: now also R37.1, U1.14 (PA0)
- net STEP_MOT_SPI_01: now also R32.1, U1.37 (PC6)
- net STEP_MOT_U1_00: now also R12.1, U1.41 (PA8)
- net STEP_MOT_U1_01: now also R9.1, U1.50 (PA15)
- net STEP_MOT_U2_00: now also R13.1, U1.56 (PB4)
- net STEP_MOT_U2_01: now also R16.1, U1.58 (PB6)
- net SWCLK: now also JS1.4 (Pin_4), R31.1, U1.49 (PA14)
- net SWDIO: now also JS1.3 (Pin_3), R30.1, U1.46 (PA13)
- net UARTTX_MOT_U1: now also DRIVER1.12 (PDN/UART), DRIVER2.12 (PDN/UART), U14.1
- net UARTTX_MOT_U2: now also DRIVER3.12 (PDN/UART), DRIVER4.12 (PDN/UART), U15.1
- net USB_D+: now also J1.A6 (DP1), J1.B6 (DP2), U1.45 (PA12), U5.2 (IOB1)
- net USB_D-: now also J1.A7 (DN1), J1.B7 (DN2), U1.44 (PA11), U5.5 (IOA2)
- net VBUS: now also D10.2 (A), J1.A4/B9 (VBUS), J1.A9/B4 (VBUS), Q1.3 (S); no longer C7.2
- net at R19.2: now also U1.16 (PA2)
- net at C20.1: now also IC1.1 (BOOT)
- net at C20.2, D2.1 (K), L1.1: now also IC1.8 (PH)
- net at TP4.1: now also FB1.1, PS1.2 (-)
- net at F1.1: now also PS1.1 (+); no longer TP5.1
- net at C17.1: now also IC1.4 (SS)
- net at R3.2, R4.1: now also IC1.5 (VSENSE)
- net at C16.1, R2.1: now also IC1.6 (COMP)
- net at R1.1: now also J1.B5 (CC2)
- net at R18.2: now also U1.42 (PA9)
- net GND: now reaches C7.1, R27.2
- net GND: now also C1.1, C13.2, C14.2, C15.2, C16.2, C17.2, C18.2, C19.2, C2.2, C21.2, C22.2, C24.2, C29.2, C3.2, C30.2, C31.2, C32.2, C33.2, C34.2, C4.2, C5.2, C6.2, D2.2 (A), D4.2 (A2), R1.2, R4.2, R5.2, R8.1, SW2.1, SW3.1 (A), Y1.2 (G), Y1.4 (G), C10.2, C11.2, C12.2, C23.2, C25.2, C26.2, C27.1, C28.2, C35.2, C36.2, C37.2, C38.1, C39.2, C40.2, C41.2, C42.2, C43.2, C44.2, C45.2, C46.2, C47.2, C48.2, C49.2, C50.2, C51.2, C52.2, C8.2, C9.2, CR2.3, DRIVER1.1 (GND), DRIVER1.11 (CLK), DRIVER1.14 (MS2), DRIVER1.15 (MS1), DRIVER1.7 (GND), DRIVER2.1 (GND), DRIVER2.11 (CLK), DRIVER2.14 (MS2), DRIVER2.7 (GND), DRIVER3.1 (GND), DRIVER3.11 (CLK), DRIVER3.14 (MS2), DRIVER3.15 (MS1), DRIVER3.7 (GND), DRIVER4.1 (GND), DRIVER4.11 (CLK), DRIVER4.14 (MS2), DRIVER4.7 (GND), DRIVER5.1 (GND), DRIVER5.11 (CLK), DRIVER5.7 (GND), DRIVER6.1 (GND), DRIVER6.11 (CLK), DRIVER6.7 (GND), FB1.2, IC1.7 (GND), J1.A1/B12 (GND), J1.A12/B1 (GND), J1.S1 (SHELL), J11.2 (Pin_2), J12.2 (Pin_2), J13.2 (Pin_2), J14.2 (Pin_2), J15.2 (Pin_2), J16.2 (Pin_2), J17.2 (Pin_2), J18.2 (Pin_2), JC1.3 (Pin_3), JC2.3 (Pin_3), JC3.3 (Pin_3), JS1.2 (Pin_2), JU1.3 (Pin_3), R29.2, R31.2, R50.2, R51.2, R52.2, R53.2, TP1.1, TP2.1, U1.12 (VSSA), U1.18 (VSS), U1.31 (VSS), U1.47 (VSS), U1.63 (VSS), U11.2 (GND), U11.8 (RS), U12.3 (GND), U12.8 (GND), U14.2, U15.2, U16.3 (GND), U18.1 (CAL_EN), U18.7 (GND), U19.1 (CAL_EN), U19.7 (GND), U2.2 (GND), U20.1 (CAL_EN), U20.7 (GND), U21.1 (CAL_EN), U21.7 (GND), U22.1 (CAL_EN), U22.7 (GND), U3.3 (GND), U3.8 (GND), U4.3 (GND), U5.1 (IOA1), U5.4 (IOB2), U6.1 (CAL_EN), U6.7 (GND)
- new net: DRIVER3.4 (B1), JM3.1 (Pin_1)
- new net: DRIVER3.5 (A1), JM3.2 (Pin_2)
- new net: DRIVER3.6 (A2), JM3.3 (Pin_3)
- new net: DRIVER3.3 (B2), JM3.4 (Pin_4)
- new net: C18.1, C19.1, D5.2 (A), D8.2 (A), L1.2, Q1.2 (G), R3.1, R53.1, TP3.1
- new net: C35.1, R22.2, R23.1
- new net: J11.3 (Pin_3), J12.3 (Pin_3), J13.3 (Pin_3), J14.3 (Pin_3), J15.3 (Pin_3), J16.3 (Pin_3), J17.3 (Pin_3), J18.3 (Pin_3), R25.2, U16.2 (IO2)
- new net: J11.4 (Pin_4), J12.4 (Pin_4), J13.4 (Pin_4), J14.4 (Pin_4), J15.4 (Pin_4), J16.4 (Pin_4), J17.4 (Pin_4), J18.4 (Pin_4), R24.2, U16.1 (IO1)
- new net: DRIVER2.10 (STEP), R9.2
- new net: DRIVER4.9 (DIR), R17.2
- new net: R44.1, U1.27 (PB1)
- new net: DRIVER1.10 (STEP), R12.2
- new net: D5.1 (K), R50.1
- new net: D6.1 (K), R51.1
- new net: DRIVER5.10 (STEP), R37.2
- new net: DRIVER5.3 (B1), JM5.3 (Pin_3)
- new net: DRIVER5.4 (B2), JM5.1 (Pin_1)
- new net: DRIVER5.5 (A1), JM5.2 (Pin_2)
- new net: DRIVER5.6 (A2), JM5.4 (Pin_4)
- new net: DRIVER5.9 (DIR), R39.2
- new net: DRIVER1.9 (DIR), R6.2
- new net: D10.1 (K), R27.1
- new net: R42.1, U1.25 (PC5)
- new net: DRIVER6.9 (DIR), R33.2
- new net: DRIVER2.9 (DIR), R10.2
- new net: C27.2, U1.30 (VCAP_1)
- new net: R45.1, U1.28 (PB2)
- new net: J1.A5 (CC1), R29.1
- new net: DRIVER3.10 (STEP), R13.2
- new net: DRIVER3.9 (DIR), R14.2
- new net: R43.1, U1.26 (PB0)
- new net: DRIVER1.3 (B2), JM1.4 (Pin_4)
- new net: DRIVER1.4 (B1), JM1.1 (Pin_1)
- new net: DRIVER1.5 (A1), JM1.2 (Pin_2)
- new net: DRIVER1.6 (A2), JM1.3 (Pin_3)
- new net: C11.1, R20.2, R21.1
- new net: D7.1 (K), R52.1
- new net: DRIVER2.4 (B1), JM2.1 (Pin_1)
- new net: DRIVER2.5 (A1), JM2.2 (Pin_2)
- new net: DRIVER2.6 (A2), JM2.3 (Pin_3)
- new net: DRIVER2.3 (B2), JM2.4 (Pin_4)
- new net: R47.1, U1.3 (PC14)
- new net: R41.1, U1.24 (PC4)
- new net: DRIVER6.4 (B2), JM6.1 (Pin_1)
- new net: DRIVER6.5 (A1), JM6.2 (Pin_2)
- new net: DRIVER6.3 (B1), JM6.3 (Pin_3)
- new net: DRIVER6.6 (A2), JM6.4 (Pin_4)
- new net: DRIVER4.4 (B1), JM4.1 (Pin_1)
- new net: DRIVER4.5 (A1), JM4.2 (Pin_2)
- new net: DRIVER4.6 (A2), JM4.3 (Pin_3)
- new net: DRIVER4.3 (B2), JM4.4 (Pin_4)
- new net: DRIVER4.10 (STEP), R16.2
- new net: R40.1, U1.20 (PA4)
- new net: R46.1, U1.2 (PC13)
- new net: DRIVER6.10 (STEP), R32.2
- new net +3V3: U18.2 (VDD), U19.2 (VDD), U20.2 (VDD), U21.2 (VDD), U22.2 (VDD), U6.2 (VDD)
- new net CAN_H LINE: C36.1, C9.1, CR2.2, JC1.2 (Pin_2), JC2.2 (Pin_2), JC3.2 (Pin_2), R20.1, R22.1, U11.7 (CANH)
- new net CAN_L LINE: C28.1, C8.1, CR2.1, JC1.1 (Pin_1), JC2.1 (Pin_1), JC3.1 (Pin_1), R21.2, R23.2, U11.6 (CANL)
- new net CS_MOT_SPI_00: DRIVER5.13 (CSN), R46.2
- new net CS_MOT_SPI_01: DRIVER6.13 (CSN), R47.2
- new net DIAG_MOT_SPI_00: DRIVER5.17 (DIAG0), R49.1, U1.57 (PB5)
- new net DIAG_MOT_SPI_01: DRIVER6.17 (DIAG0), R48.1, U1.59 (PB7)
- new net DIAG_MOT_U1_00: DRIVER1.18 (DIAG), U1.54 (PD2)
- new net DIAG_MOT_U1_01: DRIVER2.18 (DIAG)
- new net DIAG_MOT_U2_00: DRIVER3.18 (DIAG)
- new net DIAG_MOT_U2_01: DRIVER4.18 (DIAG)
- new net DIR_MOT_SPI_00: R39.1, U1.15 (PA1)
- new net DIR_MOT_SPI_01: R33.1, U1.17 (PA3)
- new net DIR_MOT_U1_00: R6.1, U1.8 (PC0)
- new net DIR_MOT_U1_01: R10.1, U1.9 (PC1)
- new net DIR_MOT_U2_00: R14.1, U1.10 (PC2)
- new net DIR_MOT_U2_01: R17.1, U1.11 (PC3)
- new net ENC1_CSN: R40.2, U6.6 (CSN)
- new net ENC2_CSN: R41.2, U18.6 (CSN)
- new net ENC3_CSN: R42.2, U19.6 (CSN)
- new net ENC4_CSN: R43.2, U20.6 (CSN)
- new net ENC5_CSN: R44.2, U21.6 (CSN)
- new net ENC6_CSN: R45.2, U22.6 (CSN)
- new net EN_MOT_SPI_00: DRIVER5.16 (~{EN}), R38.1, U1.4 (PC15)
- new net EN_MOT_SPI_01: DRIVER6.16 (~{EN}), R34.1, U1.33 (PB12)
- new net EN_MOT_U1_00: DRIVER1.16 (~{EN}), R7.1, U1.38 (PC7)
- new net EN_MOT_U1_01: DRIVER2.16 (~{EN}), R11.1, U1.39 (PC8)
- new net EN_MOT_U2_00: DRIVER3.16 (~{EN}), R15.1, U1.40 (PC9)
- new net EN_MOT_U2_01: DRIVER4.16 (~{EN}), R28.1, U1.43 (PA10)
- new net HEARTBEAT_LED: D7.2 (A), U1.55 (PB3)
- new net UARTRX_RPI: JU1.2 (Pin_2), U1.52 (PC11), U4.1 (IO1)
- new net UARTTX_RPI: JU1.1 (Pin_1), U1.51 (PC10), U4.2 (IO2)
- no-connect marks 6 -> 26
Other:
- removed sheet MOTOR_CONTROL
- note added: "5V (BUCK) VS 5V (VBUS) POWER PMOS"
- note added: "CAN"
- note added: "CAN CONNECTORS"
- note added: "ENCODER_1"
- note added: "ENCODER_2"
- note added: "ENCODER_3"
- note added: "ENCODER_4"
- note added: "ENCODER_5"
- note added: "ENCODER_6"
- note added: "I2C NETWORK"
- note added: "MAGNETIC ENCODERS"
- note added: "MCU ESSENTIALS"
- note added: "MCU LED"
- note added: "MOTOR DRIVERS"
- note added: "MOTOR UART ESD"
- note added: "POWER RAIL 24V->5V"
- note added: "RPI UART ESD"
- note added: "SERIAL WIRE DEBUG"
- note added: "SPI1 ESD"
- note added: "SPI2 ESD"
- note added: "STM32 MCU"
- note added: "STM32F446RET6 MCU"
- note added: "TMC2209 : USART1 : ADDRESS - 00"
- note added: "TMC2209 : USART1 : ADDRESS - 01"
- note added: "TMC2209 : USART2 : ADDRESS - 00"
- note added: "TMC2209 : USART2 : ADDRESS - 01"
- note added: "TMC5160 : SPI1 : USER_ADDRESS - 00"
- note added: "TMC5160 : SPI1 : USER_ADDRESS - 01"
- note added: "USB C 2.0"
- note removed: "5V/VBUS"
- title: (none) -> Arsenal - Main Board
- moved on the sheet: C1, C14, C15, C16, C17, C18, C19, C2, C20, C21, C22, C24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
